Commit message: [Enhancement] Add visual markers for panda robot fingertips

File: mani_skill/assets/robots/panda/panda_v2.urdf (robot description, URDF)
Before this commit: robot panda, 15 links, 14 joints
Links:
- added link panda_leftfinger_tip; visual sphere radius=0.005
- added link panda_rightfinger_tip; visual sphere radius=0.005
Joints:
- added joint panda_leftfinger_tip_joint: type fixed, parent panda_leftfinger, child panda_leftfinger_tip, origin xyz=0 0.00758 0.04525 rpy=0 0 0
- added joint panda_rightfinger_tip_joint: type fixed, parent panda_rightfinger, child panda_rightfinger_tip, origin xyz=0 -0.00758 0.04525 rpy=0 0 0

File: mani_skill/assets/robots/so100/so100.urdf (robot description, URDF)
Before this commit: robot SO_5DOF_ARM100_8j_URDF.SLDASM, 9 links, 8 joints
Links:
- link Fixed_Jaw_tip: geometry visual sphere radius=0.01
- link Moving_Jaw_tip: geometry visual sphere radius=0.01
